File: 655-Kicad/655.kicad_pcb (KiCad board)
At the start: 2 copper layers, 324.7 x 97.7 mm, 168 parts, among them IC1 ATMEGA32U4, J1 USBMINI_B05, P1 CONN_1, P2 CONN_1, P3 CONN_1, P4 CONN_1, P5 CONN_1, P6 CONN_1, SW0:0 F0, SW0:1 CTRL, SW0:10 CMD, SW0:11 ALT, SW0:12 CTRL, SW0:13 ←, SW0:14 ↓, SW0:15 →, SW0:2 ALT, SW0:3 CMD, SW0:7 SPACE, SW1:0 F1, SW1:1 SHIFT, SW1:10 ,, SW1:11 ., SW1:12 ?, SW1:13 SHIFT, SW1:14 ↑, SW1:15 END, SW1:3 Z, SW1:4 X, SW1:5 C, SW1:6 V, SW1:7 B, SW1:8 N, SW1:9 M, SW2:0 F2, SW2:1 CAPS, SW2:10 L, SW2:11 ;, SW2:12 ', SW2:14 ENTER, SW2:15 PGDWN, SW2:2 A, SW2:3 S, SW2:4 D, SW2:5 F, SW2:6 G, SW2:7 H, SW2:8 J, SW2:9 K, SW3:0 F3, SW3:1 TAB, SW3:10 O, SW3:11 P, SW3:12 {, SW3:13 }, SW3:14 BCKSL, SW3:15 PGUP, SW3:2 Q, SW3:3 W, SW3:4 E, SW3:5 R, SW3:6 T, SW3:7 Y, SW3:8 U, SW3:9 I, SW4:0 F4, SW4:1 TILDE, SW4:10 9, SW4:11 0, SW4:12 -, SW4:13 =, SW4:14 BCKSP, SW4:15 ESC, SW4:2 1, SW4:3 2, SW4:4 3, SW4:5 4, SW4:6 5, SW4:7 6, SW4:8 7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

Commit message: update edge cuts to fit in the case
Other:
- board size 324.7 x 97.7 mm -> 322.6 x 100 mm
Changed lines of the file:
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@@
     (area 98.945699 147.9074 423.989501 249.008901)
     (thickness 1.6002)
-    (drawings 461)
+    (drawings 456)
     (tracks 2654)
     (zones 0)
@@
       (net 20 GND))
   )
-  (gr_line (start 423.799 248.7676) (end 423.7736 248.7676) (angle 90) (layer Edge.Cuts) (width 0.381))
-  (gr_line (start 423.799 248.2596) (end 423.799 248.7676) (angle 90) (layer Edge.Cuts) (width 0.381))
-  (gr_line (start 99.1362 248.3866) (end 99.1362 248.4628) (angle 90) (layer Edge.Cuts) (width 0.381))
-  (gr_line (start 99.1362 248.8184) (end 99.1362 248.412) (angle 90) (layer Edge.Cuts) (width 0.381))
-  (gr_line (start 99.1362 248.4374) (end 99.1362 248.412) (angle 90) (layer Edge.Cuts) (width 0.381))
-  (gr_line (start 99.1362 151.11) (end 99.1362 248.3866) (angle 90) (layer Edge.Cuts) (width 0.381))
-  (gr_line (start 423.799 151.1046) (end 423.799 248.4374) (angle 90) (layer Edge.Cuts) (width 0.381))
-  (gr_line (start 423.799 248.8184) (end 99.187 248.8184) (angle 90) (layer Edge.Cuts) (width 0.381))
-  (gr_line (start 99.187 151.1046) (end 423.799 151.1046) (angle 90) (layer Edge.Cuts) (width 0.381))
+  (gr_line (start 422.9608 152.4508) (end 100.4062 152.4508) (angle 90) (layer Edge.Cuts) (width 0.381))
+  (gr_line (start 422.9608 252.4506) (end 422.9608 152.4508) (angle 90) (layer Edge.Cuts) (width 0.381))
+  (gr_line (start 100.4062 252.4506) (end 422.9608 252.4506) (angle 90) (layer Edge.Cuts) (width 0.381))
+  (gr_line (start 100.4062 152.4762) (end 100.4062 252.4506) (angle 90) (layer Edge.Cuts) (width 0.381))
   (gr_line (start 406.5542 169.4032) (end 406.5542 155.4025) (layer Eco2.User) (width 0.1))
   (gr_line (start 420.5552 169.4032) (end 406.5542 169.4032) (layer Eco2.User) (width 0.1))
