File: Test board/testboard.sch (KiCad schematic (older format))
At the start: 30 parts, among them IC1 ATMEGA32U4, J1 USBMINI_B05, P1 CONN_1, P2 CONN_1, P3 CONN_1, P4 CONN_1, P5 CONN_1, P6 CONN_1, SW0:0 F0, SW0:1 CTRL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

Commit message: Test board and full board BOM files
Parts:
- C1, C2: Link (none) -> http://www.digikey.com/product-detail/en/avx-corporation/08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
- C3, C8: Link (none) -> http://www.digikey.com/product-detail/en/yageo/CC0805KKX7R8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
- C4, C5, C6, C7: Link (none) -> http://www.digikey.com/product-detail/en/yageo/CC0805KRX7R9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
- D0:0, D0:1, D1:0, D1:1: Link (none) -> http://www.digikey.com/product-detail/en/fairchild-semicond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
- IC1: Link (none) -> http://www.digikey.com/product-detail/en/atmel/ATMEGA32U4-A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
- J1: Link (none) -> http://www.digikey.com/product-detail/en/molex-llc/06750310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
- R1, R2: Link (none) -> http://www.digikey.com/product-detail/en/yageo/RC0805JR-072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
- R3, R4: Link (none) -> http://www.digikey.com/scripts/DkSearch/dksus.dll?Detail&it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
- S0: Link (none) -> http://www.digikey.com/product-detail/en/c-k-components/KSE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
- X1: Link (none) -> http://www.digikey.com/product-detail/en/txc-corporation/9B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; Source http://www.tme.eu/en/details/hc49us-ff3f16.0000/tht-quartz-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 -> (none)

Commit message: change resistor footprints to 0805R, add caps led
Parts:
- R1, R2, R3, R4: footprint res:resistor -> 0805:0805R
Changed lines of the file:
@@
 F 0 "R1" V 3150 9300 50  0000 C CNN
 F 1 "22" V 3250 9400 50  0000 C CNN
-F 2 "res:resistor" V 3180 9400 50  0001 C CNN
+F 2 "0805:0805R" V 3180 9400 50  0001 C CNN
 F 3 "" H 3250 9400 50  0000 C CNN
 F 4 "http://www.digikey.com/product-detail/en/yageo/RC0805JR-0722RL/311-22ARCT-ND/731232" V 3250 9400 60  0001 C CNN "Link"
@@
 F 0 "R2" V 3350 9400 50  0000 C CNN
 F 1 "22" V 3250 9500 50  0000 C CNN
-F 2 "res:resistor" V 3180 9500 50  0001 C CNN
+F 2 "0805:0805R" V 3180 9500 50  0001 C CNN
 F 3 "" H 3250 9500 50  0000 C CNN
 F 4 "http://www.digikey.com/product-detail/en/yageo/RC0805JR-0722RL/311-22ARCT-ND/731232" V 3250 9500 60  0001 C CNN "Link"
@@
 F 0 "R4" V 4230 6150 50  0000 C CNN
 F 1 "10k" V 4150 6150 50  0000 C CNN
-F 2 "res:resistor" V 4080 6150 50  0001 C CNN
+F 2 "0805:0805R" V 4080 6150 50  0001 C CNN
 F 3 "" H 4150 6150 50  0000 C CNN
 F 4 "http://www.digikey.com/scripts/DkSearch/dksus.dll?Detail&itemSeq=205254129&uq=636075607746610083" V 4150 6150 60  0001 C CNN "Link"
@@
 F 0 "R3" V 6980 10650 50  0000 C CNN
 F 1 "10k" V 6900 10650 50  0000 C CNN
-F 2 "res:resistor" V 6830 10650 50  0001 C CNN
+F 2 "0805:0805R" V 6830 10650 50  0001 C CNN
 F 3 "" H 6900 10650 50  0000 C CNN
 F 4 "http://www.digikey.com/scripts/DkSearch/dksus.dll?Detail&itemSeq=205254129&uq=636075607746610083" V 6900 10650 60  0001 C CNN "Link"
